File: KiCad_Project/mHz_oscillator.kicad_sch (KiCad schematic)
At the start: 111 parts, among them J1 Saw, J2 Trigger, J3 Triangle, J4 CV_in, J5 Sinus, J6 PWM, J7 Conn_02x08_Odd_Even, Q1 BC847, Q2 BC847, SW1 One Shot or Continous, SW2 Trigger Button, SW3 Freq Range, U1 LM324, U2 LM324, U3 LM324, U4 LM324, U5 LM324, U6 4013, U7 4071, U8 LM311

Commit message: added interface and main pcb schematics
Parts:
- removed C1: 69n, Capacitor_SMD:C_1206_3216Metric, symbol Device:C_Small
- removed C10, C11, C12, C13, C14, C15, C16, C17, C18, C19, C3, C4, C6, C8, C9: 100n, Capacitor_SMD:C_1206_3216Metric, symbol Device:C_Small
- removed C2: 470n, Capacitor_SMD:C_1206_3216Metric, symbol Device:C_Small
- removed C5, C7: 47n, Capacitor_SMD:C_1206_3216Metric, symbol Device:C_Small
- removed D1, D3, D4, D5, D8: 1N4148, Diode_SMD:D_1206_3216Metric, symbol Device:D_Small
- removed D10, D11: 1N4148, Diode_SMD:D_1206_3216Metric, symbol Device:D
- removed D2, D6, D7, D9: Blue, LED_THT:LED_D3.0mm, symbol Device:LED_Small
- removed J1: Saw, component-library:Jack_3.5mm_VERTICAL, symbol Connector:AudioJack3
- removed J2: Trigger, component-library:Jack_3.5mm_VERTICAL, symbol Connector:AudioJack3
- removed J3: Triangle, component-library:Jack_3.5mm_VERTICAL, symbol Connector:AudioJack3
- removed J4: CV_in, component-library:Jack_3.5mm_VERTICAL, symbol Connector:AudioJack3
- removed J5: Sinus, component-library:Jack_3.5mm_VERTICAL, symbol Connector:AudioJack3
- removed J6: PWM, component-library:Jack_3.5mm_VERTICAL, symbol Connector:AudioJack3
- removed J7: Conn_02x08_Odd_Even, Connector_IDC:IDC-Header_2x08_P2.54mm_Vertical, symbol Connector_Generic:Conn_02x08_Odd_Even
- removed Q1, Q2: BC847, Package_TO_SOT_SMD:SOT-23, symbol Transistor_BJT:BC847
- removed R1, R12, R13, R35, R36, R37, R40, R41, R43, R48, R49, R51, R52, R7: 10k, Resistor_SMD:R_1206_3216Metric, symbol Device:R
- removed R10: 1k, Resistor_SMD:R_1206_3216Metric, symbol Device:R
- removed R11, R25, R29, R39: 3k3, Resistor_SMD:R_1206_3216Metric, symbol Device:R
- removed R14: 43k, Resistor_SMD:R_1206_3216Metric, symbol Device:R
- removed R15, R22, R23, R27, R28, R34, R45, R5, R50, R6, R8, R9: 100k, Resistor_SMD:R_1206_3216Metric, symbol Device:R
- removed R16, R2, R32, R42: 2k7, Resistor_SMD:R_1206_3216Metric, symbol Device:R
- removed R17, R53: 22k, Resistor_SMD:R_1206_3216Metric, symbol Device:R
- removed R18, R21: 1meg, Resistor_SMD:R_1206_3216Metric, symbol Device:R
- removed R19, R33, R4, R44: 860k, Resistor_SMD:R_1206_3216Metric, symbol Device:R
- removed R20: 180k, Resistor_SMD:R_1206_3216Metric, symbol Device:R
- removed R24: 56k, Resistor_SMD:R_1206_3216Metric, symbol Device:R
- removed R26: 12k, Resistor_SMD:R_1206_3216Metric, symbol Device:R
- removed R3: 150k, Resistor_SMD:R_1206_3216Metric, symbol Device:R
- removed R30, R47: 33k, Resistor_SMD:R_1206_3216Metric, symbol Device:R
- removed R31: 47k, Resistor_SMD:R_1206_3216Metric, symbol Device:R
- removed R38: 27k, Resistor_SMD:R_1206_3216Metric, symbol Device:R
- removed R46: 3k9, Resistor_SMD:R_1206_3216Metric, symbol Device:R
- removed RV1: 100k log, Potentiometer_THT:Potentiometer_Alps_RK09K_Single_Vertical, symbol Device:R_Potentiometer
- removed RV2: 10k, Potentiometer_SMD:Potentiometer_Bourns_TC33X_Vertical, symbol Device:R_Potentiometer_Trim
- removed RV3: 100k lin, Potentiometer_THT:Potentiometer_Alps_RK09K_Single_Vertical, symbol Device:R_Potentiometer
- removed RV4, RV5, RV6, RV7: 100k, Potentiometer_SMD:Potentiometer_Bourns_TC33X_Vertical, symbol Device:R_Potentiometer_Trim
- removed SW1: One Shot or Continous, symbol Switch:SW_SPDT
- removed SW2: Trigger Button, symbol Switch:SW_Push
- removed SW3: Freq Range, symbol Switch:SW_SPDT
- removed TP1: -300mV, symbol Connector:TestPoint
- removed U1, U2, U3, U4, U5: LM324, Package_SO:SOIC-14_3.9x8.7mm_P1.27mm, symbol Amplifier_Operational:LM324
- removed U6: 4013, Package_SO:SOIC-14_3.9x8.7mm_P1.27mm, symbol 4xxx:4013
- removed U7: 4071, Package_SO:SOIC-14_3.9x8.7mm_P1.27mm, symbol 4xxx:4071
- removed U8: LM311, Package_SO:SOIC-8_3.9x4.9mm_P1.27mm, symbol Comparator:LM311
- added J1, J3, J5: Conn_01x06_Male, Connector_PinHeader_2.54mm:PinHeader_1x06_P2.54mm_Vertical, symbol Connector:Conn_01x06_Male
- added J10, J8: Conn_01x05_Female, Connector_PinSocket_2.54mm:PinSocket_1x05_P2.54mm_Vertical, symbol Connector:Conn_01x05_Female
- added J2, J4, J6: Conn_01x06_Female, Connector_PinSocket_2.54mm:PinSocket_1x06_P2.54mm_Vertical, symbol Connector:Conn_01x06_Female
- added J7, J9: Conn_01x05_Male, Connector_PinHeader_2.54mm:PinHeader_1x05_P2.54mm_Vertical, symbol Connector:Conn_01x05_Male
Connections:
- new net interface_pcb/0V: J5.6 (Pin_6)
- new net interface_pcb/CV_in: J9.1 (Pin_1)
- new net interface_pcb/Freq_CCW: J9.4 (Pin_4)
- new net interface_pcb/Freq_CW: J9.5 (Pin_5)
- new net interface_pcb/Freq_High: J5.2 (Pin_2)
- new net interface_pcb/Freq_Low: J5.3 (Pin_3)
- new net interface_pcb/Freq_Switch_Output: J5.1 (Pin_1)
- new net interface_pcb/Freq_Wiper: J9.3 (Pin_3)
- new net interface_pcb/PWM_CCW: J7.4 (Pin_4)
- new net interface_pcb/PWM_CW: J7.5 (Pin_5)
- new net interface_pcb/PWM_Wiper: J7.3 (Pin_3)
- new net interface_pcb/PushButton_1: J7.1 (Pin_1)
- new net interface_pcb/PushButton_2: J7.2 (Pin_2)
- new net interface_pcb/SMTS_OneShot: J5.4 (Pin_4)
- new net interface_pcb/SMTS_Output: J5.5 (Pin_5)
- new net interface_pcb/Saw: J3.3 (Pin_3)
- new net interface_pcb/Saw_LEDAnode: J3.1 (Pin_1)
- new net interface_pcb/Saw_LEDCathode: J3.2 (Pin_2)
- new net interface_pcb/Sine: J1.6 (Pin_6)
- new net interface_pcb/Sine_LEDAnode: J1.4 (Pin_4)
- new net interface_pcb/Sine_LEDCathode: J1.5 (Pin_5)
- new net interface_pcb/Square: J3.6 (Pin_6)
- new net interface_pcb/Square_LEDAnode: J3.4 (Pin_4)
- new net interface_pcb/Square_LEDCathode: J3.5 (Pin_5)
- new net interface_pcb/Triangle: J1.3 (Pin_3)
- new net interface_pcb/Triangle_LEDAnode: J1.1 (Pin_1)
- new net interface_pcb/Triangle_LEDCathode: J1.2 (Pin_2)
- new net interface_pcb/Trigger_input: J9.2 (Pin_2)
- new net main_pcb/0V: J6.6 (Pin_6)
- new net main_pcb/CV_in: J10.1 (Pin_1)
- new net main_pcb/Freq_CCW: J10.4 (Pin_4)
- new net main_pcb/Freq_CW: J10.5 (Pin_5)
- new net main_pcb/Freq_High: J6.2 (Pin_2)
- new net main_pcb/Freq_Low: J6.3 (Pin_3)
- new net main_pcb/Freq_Switch_Output: J6.1 (Pin_1)
- new net main_pcb/Freq_Wiper: J10.3 (Pin_3)
- new net main_pcb/PWM_CCW: J8.4 (Pin_4)
- new net main_pcb/PWM_CW: J8.5 (Pin_5)
- new net main_pcb/PWM_Wiper: J8.3 (Pin_3)
- new net main_pcb/PushButton_1: J8.1 (Pin_1)
- new net main_pcb/PushButton_2: J8.2 (Pin_2)
- new net main_pcb/SMTS_OneShot: J6.4 (Pin_4)
- new net main_pcb/SMTS_Output: J6.5 (Pin_5)
- new net main_pcb/Saw: J4.3 (Pin_3)
- new net main_pcb/Saw_LEDAnode: J4.1 (Pin_1)
- new net main_pcb/Saw_LEDCathode: J4.2 (Pin_2)
- new net main_pcb/Sine: J2.6 (Pin_6)
- new net main_pcb/Sine_LEDAnode: J2.4 (Pin_4)
- new net main_pcb/Sine_LEDCathode: J2.5 (Pin_5)
- new net main_pcb/Square: J4.6 (Pin_6)
- new net main_pcb/Square_LEDAnode: J4.4 (Pin_4)
- new net main_pcb/Square_LEDCathode: J4.5 (Pin_5)
- new net main_pcb/Triangle: J2.3 (Pin_3)
- new net main_pcb/Triangle_LEDAnode: J2.1 (Pin_1)
- new net main_pcb/Triangle_LEDCathode: J2.2 (Pin_2)
- new net main_pcb/Trigger_input: J10.2 (Pin_2)
- no-connect marks 18 -> 0
Other:
- added sheet interface_pcb (interface_pcb.kicad_sch)
- added sheet main_pcb (main_pcb.kicad_sch)
- note removed: "LED Bias and Buffers"
- note removed: "PWM/Square Generator"
- note removed: "Power"
- note removed: "Saw to Triangle Shaper"
- note removed: "Sawtooth Core"
- note removed: "Sine Shaper"
- note removed: "Trigger Circiut"
